File: Karman Eagle/Karman Projects/Dev Board/Current/Rev 1/Dev Board.sch (EAGLE design)
At the start: 39 parts, among them J1 I2C1, J10 P8-P13, J2 P0-P3, J3 A0-A3, J5 P4-P7, J6 VCC, J7 GND, J8 SPI1, J9 UART5, U1 BNO055, U2 ADXL377, U3 BNO055

Commit message: 5/13/19 Dev board update
Parts:
- added C17, C19, C23, C29, C31: 100nF, CGA3E2X7R1H104K080AD:CGA3E2X7R1H104K080AD
- added C18, C20, C24, C30, C32: 4.7uF, CGA3E2X7R1H104K080AD:CGA3E2X7R1H104K080AD
- added C25, C26: 2.2uF, CGA3E2X7R1H104K080AD:CGA3E2X7R1H104K080AD
- added J11: 47219-2001, 47219-2001:47219-2001
- added J4: Debug, SparkFun-Connectors:CONN_04
- added U$4: (no value), Molex:087831-0819
Connections:
- removed net ST_PF3: U2.ST
- removed net XOUT_PA3: C16.1, U$1.PA3, U2.XOUT
- removed net YOUT_PC0: C15.1, U$1.PC0, U2.YOUT
- removed net ZOUT_PC3: C8.1, U$1.PC3, U2.ZOUT
- new net CS2_PB12: U$1.PB12, U$4.7
- new net CS4_PE3: J11.CD/DAT3(CS), U$1.PE3
- new net MISO2_PB14: U$1.PB14, U$4.6
- new net MISO4_PE5: J11.DAT0(MISO), U$1.PE5
- new net MOSI2_PB15: U$1.PB15, U$4.2
- new net MOSI4_PE6: J11.CMD(MOSI), U$1.PE6
- new net N$2: C17.1, C18.1, C19.1, C20.1, C23.1, C24.1, C29.1, C30.1, C31.1, C32.1
- new net N$4: C25.1, U$1.VCAP2
- new net N$7: C26.2, U$1.VCAP1
- new net RX7_PE7: U$1.PE7, U$4.1
- new net SCL2_PB13: U$1.PB13, U$4.3
- new net SCL4_PE2: J11.CLK, U$1.PE2
- new net ST_PC3: U$1.PC3, U2.ST
- new net SWDIO_PA13: J4.1, U$1.PA13
- new net SWSLK_PA14: J4.2, U$1.PA14
- new net TX7_PE8: U$1.PE8, U$4.5
- new net XOUT_PC0: C16.1, U$1.PC0, U2.XOUT
- new net YOUT_PC1: C15.1, U$1.PC1, U2.YOUT
- new net ZOUT_PC2: C8.1, U$1.PC2, U2.ZOUT
- net 3V3: now also J11.VDD, J4.3, U$1.VDD@1, U$1.VDD@2, U$1.VDD@3, U$1.VDD@4, U$1.VDD@5, U$4.4
- net A0_PA1: now also U$1.PA1
- net A1_PA2: now also U$1.PA2
- net A2_PA3: now also U$1.PA3
- net GND: now also C17.2, C18.2, C19.2, C20.2, C23.2, C24.2, C25.2, C26.1, C29.2, C30.2, C31.2, C32.2, J11.GND@1, J11.GND@2, J11.GND@3, J11.GND@4, J11.VSS, J4.4, U$1.VSS@1, U$1.VSS@2, U$1.VSS@3, U$1.VSS@4, U$1.VSS@5, U$4.8
- net RX5_PD0: now also U$1.PD0
- net TX5_PD1: now also U$1.PD1
Other:
- note added: "Breakout Pins"
- note added: "GPS/Radio Module"
- note added: "IMU 2"
- note added: "MCU Power Supply"
- note added: "MicroSD"
- note added: "Place near pin 100"
- note added: "Place near pin 11"
- note added: "Place near pin 27"
- note added: "Place near pin 50"
- note added: "Place near pin 75"

Commit message: 5/13/19 10:08PM Dev board update
Parts:
- added C21, C22: 10 uF, CGA3E2X7R1H104K080AD:CGA3E2X7R1H104K080AD
- added R5: 121Ω, CRGH0603F221K:CRGH0603F221K
- added R6: 5kΩ, CRGH0603F221K:CRGH0603F221K
- added U$6: LM1085, LM1085:LM1085
Connections:
- removed net N$2: C17.1, C18.1, C19.1, C20.1, C23.1, C24.1, C29.1, C30.1, C31.1, C32.1
- new net N$10: C17.1, C18.1, C19.1, C20.1, C22.1, C23.1, C24.1, C29.1, C30.1, C31.1, C32.1, R5.1, U$6.VO
- new net N$8: R5.2, R6.2, U$6.ADJ
- new net N$9: C21.2, C22.2, R6.1
- net 3V3: now also C21.1, U$6.VI

Commit message: 5/24/19 20:26 PCB Update
Connections:
- net 3V3: now also U$1.VDDA
- net GND: now also U$1.VSSA
Changed lines of the file:
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@@
 <part name="R6" library="CRGH0603F221K" deviceset="CRGH0603F221K" device="" value="5kΩ"/>
 <part name="GND30" library="SparkFun-PowerSymbols" library_urn="urn:adsk.eagle:library:530" deviceset="GND" device=""/>
+<part name="GND35" library="SparkFun-PowerSymbols" library_urn="urn:adsk.eagle:library:530" deviceset="GND" device=""/>
 </parts>
 <sheets>
@@
 <attribute name="VALUE" x="58.42" y="181.356" size="1.778" layer="96" align="top-center"/>
 </instance>
+<instance part="GND35" gate="1" x="10.16" y="91.44" smashed="yes" rot="R270">
+<attribute name="VALUE" x="9.906" y="91.44" size="1.778" layer="96" rot="R270" align="top-center"/>
+</instance>
 </instances>
 <busses>
@@
 <wire x1="194.31" y1="149.86" x2="194.31" y2="148.59" width="0.1524" layer="91"/>
 </segment>
+<segment>
+<pinref part="U$1" gate="G$1" pin="VSSA"/>
+<wire x1="22.86" y1="92.71" x2="12.7" y2="92.71" width="0.1524" layer="91"/>
+<pinref part="GND35" gate="1" pin="GND"/>
+<wire x1="12.7" y1="92.71" x2="12.7" y2="91.44" width="0.1524" layer="91"/>
+</segment>
 </net>
 <net name="SCL1_PB8" class="0">
@@
 <junction x="43.18" y="205.74"/>
 </segment>
+<segment>
+<pinref part="U$1" gate="G$1" pin="VDDA"/>
+<wire x1="22.86" y1="87.63" x2="19.05" y2="87.63" width="0.1524" layer="91"/>
+<label x="19.05" y="87.63" size="1.016" layer="95" rot="R180" xref="yes"/>
+</segment>
 </net>

Commit message: 5/25/19 11:45 PCB Issued for Review
Parts:
- added C27: 22uF, CGA3E2X7R1H104K080AD:CGA3E2X7R1H104K080AD
- added C28: 1uF, CGA3E2X7R1H104K080AD:CGA3E2X7R1H104K080AD
- added C33: 10nF, CGA3E2X7R1H104K080AD:CGA3E2X7R1H104K080AD
- added C34: 4.7nF, CGA3E2X7R1H104K080AD:CGA3E2X7R1H104K080AD
- added J12: 105164-0001, 105164-0001:105164-0001
- added L1: 2.2uH, 0603_Inductor:MLF1608E100J
- added R7: 59k, 0603_Resistor:CRGH0603F221K
- added R8: 42.2k, 0603_Resistor:CRGH0603F221K
- added U$10, U$11, U$7, U$8, U$9: PESD3V3S1UL, PESD3V3S1UL:PESD3V3S1UL
- R5: value 121Ω -> 100k; device CRGH0603F221K:CRGH0603F221K -> 0603_Resistor:CRGH0603F221K
- R6: value 5kΩ -> 1M; device CRGH0603F221K:CRGH0603F221K -> 0603_Resistor:CRGH0603F221K
- U$6: value LM1085 -> TPS62172; device LM1085:LM1085 -> TPS62172:TPS62172
Connections:
- removed net N$9: C21.2, C22.2, R6.1
- new net N$13: J12.ID
- new net N$14: C34.2, J12.SHIELD, R6.1, U$10.CA, U$11.CA, U$9.CA
- new net PG_PD7: R5.1, U$1.PD7, U$6.PG
- new net USBD+_PB3: J12.D+, U$1.PB3, U$11.AN, U$8.CA
- new net USBD-_PB4: J12.D-, U$1.PB4, U$10.AN, U$7.CA
- new net USBSENSE_PB5: R7.2, R8.1, U$1.PB5
- new net VIN: C21.1, J12.5V_IN, R8.2, U$6.EN, U$6.VIN, U$7.AN, U$8.AN, U$9.AN
- net 3V3: now also C22.2, C27.2, C28.2, C33.2, L1.2, R5.2, U$1.VREF+, U$6.VOS; no longer C21.1, U$6.VI
- net GND: now also C21.2, C27.1, C28.1, C33.1, C34.1, J12.GND, R6.2, R7.1, U$6.AGND, U$6.FB, U$6.PGND, U$6.THERMAL_PAD
- net N$10: no longer R5.1, U$6.VO
- net N$8: now also L1.1, U$6.SW; no longer R5.2, R6.2, U$6.ADJ
Other:
- note added: "3V3 Plane Regulator"
- note added: "Micro USB"
- moved on the sheet: C17, C18, C19, C20, C21, C22, C23, C24, C25, C26, C29, C30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

Commit message: 5/25/19 12:47 PCB ISSUED FOR REVIEW
Other:
- moved on the sheet: J1, J10, J11, J2, J3, J4, J5, J6, J7, J8, J9, U$4

Commit message: BOM added
Parts:
- added U$13: TSX-3225, TSX-3225 16.0000MF09Z-AC0:TSX-3225
- renumbered J11 to J43
