File: Karman Eagle/Karman Projects/Dev Board/Current/Rev 1/1906152158-Dev Board.brd (EAGLE design)
At the start: 64.8 x 38.1 mm, 72 parts, among them J1 I2C1, J10 P8-P13, J12 105164-0001, J2 P0-P3, J3 A0-A3, J4 Debug, J43 47219-2001, J5 P4-P7, J6 VCC, J7 GND, J8 SPI1, J9 UART5, U1 BNO055, U2 ADXL377, U20 PESD3V3S1UL, U22 PESD3V3S1UL, U23 PESD3V3S1UL, U24 PESD3V3S1UL, U3 BNO055, U4 MS5607-02BA03, U5 MS5607-02BA03, U6 TSX-3225, U7 TPS62172, U8 STM32F767VIT6

Commit message: DevBoard update 8/2/2019 11:59PM
Parts:
- removed C22: 10 uF, CGA3E2X7R1H104K080AD:CAPC1608X95N
- added C35, C36: 8pF, CGA3E2X7R1H104K080AD:CAPC1608X95N
- added J13: VIN, SparkFun-Connectors:1X01
- added J16: Header 3x2, SparkFun-Connectors:2X3
- added R13: (no value), 0603_Resistor:RESC1608X50N
- moved J43 115.5 mm to (-72.4, 2.29), flipped to the top, turned to 0 degrees
- moved C10 113.3 mm to (50.3, 25.4), turned to 180 degrees
- moved U6 112.1 mm to (18.5, 18.0), turned to 90 degrees
- moved C9 110.0 mm to (50.3, 18.3), turned to 180 degrees
- moved U7 102.8 mm to (4.83, 2.03)
- moved R2 86.8 mm to (9.14, 13.7)
- moved R1 82.6 mm to (9.14, 15.5)
- moved C11 74.1 mm to (5.33, 26.9), turned to 180 degrees
- moved R12 72.0 mm to (9.14, 20.6)
- moved R11 67.8 mm to (9.14, 22.4)
- moved R10 63.7 mm to (9.14, 24.1)
- moved C6 62.7 mm to (10.7, 34.5)
- moved C2 62.6 mm to (2.03, 16.5)
- moved C12 60.8 mm to (2.03, 26.9)
- moved R9 59.6 mm to (9.14, 25.9)
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Connections:
- removed net N$10: C17.1, C18.1, C19.1, C20.1, C22.1, C23.1, C24.1, C29.1, C30.1, C31.1, C32.1
- new net N$15: C35.1, R13.1, U6.3
- new net N$17: J16.5
- new net N$18: C21.1, J16.2, J16.4, J16.6, U7.2, U7.3
- new net OSC_IN: R13.2, U8.12
- new net OSC_OUT: C36.2, U6.1, U8.13
- new net USB_5V: J12.1, J16.3, R8.2, U20.2, U22.2
- net 3V3: now also C1.2, C17.1, C18.1, C19.1, C2.2, C20.1, C23.1, C24.1, C29.1, C30.1, C31.1, C32.1, C4.2, R1.2, R2.2, R3.2, R4.2, U1.28, U1.3; no longer C22.2
- net GND: now also C35.2, C36.1, U6.2, U6.4
- net NRESET: now also U8.14
- net VDD: no longer C4.2, U1.3
- net VDDIO: no longer C1.2, C2.2, R1.2, R2.2, R3.2, R4.2, U1.28
- net VIN: now also J13.1, J16.1; no longer C21.1, J12.1, R8.2, U20.2, U22.2, U7.2, U7.3
Routing:
- net GND: track 0.00 -> 88.9 mm, vias 0 -> 54
- net 3V3: track 0.00 -> 48.7 mm
- net P13_PC9: track 0.00 -> 24.3 mm
- net P12_PC8: track 0.00 -> 21.4 mm
- net P11_PC7: track 0.00 -> 18.9 mm
- net P8_PD14: track 0.00 -> 16.8 mm
- net P10_PC6: track 0.00 -> 16.5 mm
- net P9_PD15: track 0.00 -> 16.1 mm
- net VDDIO: track 0.00 -> 16.1 mm
- net PIN7: track 0.00 -> 14.5 mm, vias 0 -> 2
- net PIN8: track 0.00 -> 13.4 mm, vias 0 -> 2
- net BL_IND: track 0.00 -> 12.7 mm, vias 0 -> 2
- net PIN24: track 0.00 -> 12.1 mm, vias 0 -> 2
- net OSC_OUT: track 0.00 -> 9.80 mm
- net PIN23: track 0.00 -> 9.47 mm, vias 0 -> 2
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Other:
- board size 64.8 x 38.1 mm -> 81.3 x 38.1 mm
- board text added: "Via drill: 0.3mm Via Hole: Auto"
