File: Karman Eagle/Karman Projects/Dev Board/Current/Rev 1/1906152158-Dev Board.sch (EAGLE design)
At the start: 72 parts, among them J1 I2C1, J10 P8-P13, J12 105164-0001, J2 P0-P3, J3 A0-A3, J4 Debug, J43 47219-2001, J5 P4-P7, J6 VCC, J7 GND, J8 SPI1, J9 UART5, U1 BNO055, U2 ADXL377, U20 PESD3V3S1UL, U22 PESD3V3S1UL, U23 PESD3V3S1UL, U24 PESD3V3S1UL, U3 BNO055, U4 MS5607-02BA03, U5 MS5607-02BA03, U6 TSX-3225, U7 TPS62172, U8 STM32F767VIT6

Commit message: DevBoard update 8/2/2019 11:59PM
Parts:
- removed C22: 10 uF, CGA3E2X7R1H104K080AD:CGA3E2X7R1H104K080AD
- added C35, C36: 8pF, CGA3E2X7R1H104K080AD:CGA3E2X7R1H104K080AD
- added J13: VIN, SparkFun-Connectors:CONN_01
- added J16: Header 3x2, SparkFun-Connectors:CONN_03X22X3_SILK_MALE_PTH
- added R13: (no value), 0603_Resistor:CRGH0603F221K
Connections:
- removed net N$10: C17.1, C18.1, C19.1, C20.1, C22.1, C23.1, C24.1, C29.1, C30.1, C31.1, C32.1
- new net N$15: C35.1, R13.1, U6.3
- new net N$17: J16.5
- new net N$18: C21.1, J16.2, J16.4, J16.6, U7.EN, U7.VIN
- new net OSC_IN: R13.2, U8.PH0-OSC_IN
- new net OSC_OUT: C36.2, U6.1, U8.PH1-OSC_OUT
- new net USB_5V: J12.5V_IN, J16.3, R8.2, U20.AN, U22.AN
- net 3V3: now also C1.2, C17.1, C18.1, C19.1, C2.2, C20.1, C23.1, C24.1, C29.1, C30.1, C31.1, C32.1, C4.2, R1.2, R2.2, R3.2, R4.2, U1.VDD@1, U1.VDDIO; no longer C22.2
- net GND: now also C35.2, C36.1, U6.GND@1, U6.GND@2
- net NRESET: now also U8.NRST
- net VDD: no longer C4.2, U1.VDD@1
- net VDDIO: no longer C1.2, C2.2, R1.2, R2.2, R3.2, R4.2, U1.VDDIO
- net VIN: now also J13.1, J16.1; no longer C21.1, J12.5V_IN, R8.2, U20.AN, U22.AN, U7.EN, U7.VIN
Other:
- note added: "CRYSTAL"
- note added: "Headers"
- note added: "Power Source Select"
- note removed: "Breakout Pins"
