File: Karman Eagle/Karman Projects/Dev Board/Current/Rev 1/1908011900-Dev Board.brd (EAGLE design)
At the start: 77.5 x 25.9 mm, 88 parts, among them J1 I2C1, J10 P8-P13, J12 105164-0001, J13 VIN, J16 Header 3x2, J2 P0-P3, J3 A0-A3, J4 Debug, J43 47219-2001, J5 P4-P7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

Commit message: Just some Eagle files that I never committed
Parts:
- C35, C36: value 8pF -> 4pF
Changed lines of the file:
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@@
 <?xml version="1.0" encoding="utf-8"?>
 <!DOCTYPE eagle SYSTEM "eagle.dtd">
-<eagle version="9.4.2">
+<eagle version="9.5.0">
 <drawing>
 <settings>
-<setting alwaysvectorfont="yes"/>
+<setting alwaysvectorfont="no"/>
 <setting verticaltext="up"/>
 </settings>
@@
 <layer number="115" name="ReferenceISLANDS" color="7" fill="1" visible="no" active="yes"/>
 <layer number="116" name="Patch_BOT" color="9" fill="4" visible="no" active="yes"/>
+<layer number="117" name="noPrintText" color="7" fill="1" visible="no" active="yes"/>
 <layer number="118" name="Rect_Pads" color="7" fill="1" visible="no" active="yes"/>
 <layer number="119" name="LOGOS" color="7" fill="1" visible="no" active="yes"/>
@@
 <attribute name="NAME" x="37.874" y="19.911" size="0.8" layer="25"/>
 </element>
-<element name="C35" library="CGA3E2X7R1H104K080AD" package="CAPC1608X95N" value="8pF" x="29.718" y="14.478" smashed="yes" rot="R90">
+<element name="C35" library="CGA3E2X7R1H104K080AD" package="CAPC1608X95N" value="4pF" x="29.718" y="14.478" smashed="yes" rot="R90">
 <attribute name="AVAILABILITY" value="Unavailable" x="29.718" y="14.478" size="1.778" layer="27" rot="R90" display="off"/>
 <attribute name="DESCRIPTION" value=" CGA Series 0603 0.1 uF 50 V ±10% X7R SMT Multilayer Ceramic Capacitor " x="29.718" y="14.478" size="1.778" layer="27" rot="R90" display="off"/>
@@
 <attribute name="PRICE" value="None" x="29.718" y="14.478" size="1.778" layer="27" rot="R90" display="off"/>
 </element>
-<element name="C36" library="CGA3E2X7R1H104K080AD" package="CAPC1608X95N" value="8pF" x="29.718" y="11.176" smashed="yes" rot="R270">
+<element name="C36" library="CGA3E2X7R1H104K080AD" package="CAPC1608X95N" value="4pF" x="29.718" y="11.176" smashed="yes" rot="R270">
 <attribute name="AVAILABILITY" value="Unavailable" x="29.718" y="11.176" size="1.778" layer="27" rot="R270" display="off"/>
 <attribute name="DESCRIPTION" value=" CGA Series 0603 0.1 uF 50 V ±10% X7R SMT Multilayer Ceramic Capacitor " x="29.718" y="11.176" size="1.778" layer="27" rot="R270" display="off"/>
